File: pcb/keyboard.kicad_pcb (KiCad board)
At the start: 4 copper layers, 191 parts, among them K1 KEYSW, K10 KEYSW, K11 KEYSW, K12 KEYSW, K13 KEYSW, K14 KEYSW, K15 KEYSW, K16 KEYSW, K17 KEYSW, K18 KEYSW, K19 KEYSW, K2 KEYSW, K20 KEYSW, K21 KEYSW, K22 KEYSW, K23 KEYSW, K24 KEYSW, K25 KEYSW, K26 KEYSW, K27 KEYSW, K28 KEYSW, K29 KEYSW, K3 KEYSW, K30 KEYSW, K31 KEYSW, K32 KEYSW, K33 KEYSW, K34 KEYSW, K35 KEYSW, K36 KEYSW, K37 KEYSW, K38 KEYSW, K39 KEYSW, K4 KEYSW, K40 KEYSW, K41 KEYSW, K42 KEYSW, K43 KEYSW, K45 KEYSW, K46 KEYSW, K47 KEYSW, K48 KEYSW, K49 KEYSW, K5 KEYSW, K50 KEYSW, K51 KEYSW, K52 KEYSW, K53 KEYSW, K54 KEYSW, K55 KEYSW, K56 KEYSW, K57 KEYSW, K58 KEYSW, K59 KEYSW, K6 KEYSW, K60 KEYSW, K61 KEYSW, K62 KEYSW, K63 KEYSW, K67 KEYSW, K7 KEYSW, K70 KEYSW, K71 KEYSW, K72 KEYSW, K73 KEYSW, K74 KEYSW, K75 KEYSW, K8 KEYSW, K9 KEYSW, Q1 FDN340P, Q2 FS8025A, Q3 FDN340P, U1 nRF52840, U2 TP4056-42-ESOP8, U3 DW01A, X1 32MHz

Commit message: Place all keys
Parts:
- moved K15 301.1 mm to (342.9, 109.5)
- moved K30 282.4 mm to (342.9, 128.6)
- moved K13 247.3 mm to (285.8, 109.5)
- moved K28 234.8 mm to (295.3, 128.6)
- moved K12 232.7 mm to (266.7, 109.5)
- moved K45 225.0 mm to (342.9, 147.6)
- moved K11 219.9 mm to (247.7, 109.5)
- moved K27 217.0 mm to (276.2, 128.6)
- moved K10 209.2 mm to (228.6, 109.5)
- moved K26 200.6 mm to (257.2, 128.6)
- moved K43 194.6 mm to (300.0, 147.6)
- moved K9 186.9 mm to (209.6, 109.5)
- moved K25 185.9 mm to (238.1, 128.6)
- moved K24 173.6 mm to (219.1, 128.6)
- moved K8 165.2 mm to (190.5, 109.5)
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
Commit message: Fix some labels
Parts:
- moved U1 107.5 mm to (307.2, 79.2)
- moved BT1 79.5 mm to (180.2, 85.2)
- turned K12 to 90 degrees
- turned K13 to 90 degrees

Commit message: tinkering >:3
Parts:
- added J3: Conn_Coaxial, Connector_Coaxial:SMA_Molex_73251-1153_EdgeMount_Horizontal, F.Cu at (255.5, 61.3)
- D1, D10, D11, D12, D13, D14, D15, D2, D3, D4, D5, D6, D7, D8, D9: moved to B.Cu
- moved D16 358.9 mm to (24.8, 128.9)
- moved D17 358.9 mm to (24.8, 132.0)
- moved D18 358.9 mm to (24.8, 135.0)
- moved D19 358.9 mm to (24.8, 138.0)
- moved D20 358.9 mm to (24.8, 141.1)
- moved D21 358.9 mm to (24.8, 144.1)
- moved D22 358.9 mm to (24.8, 147.2)
- moved D23 358.9 mm to (24.8, 150.2)
- moved D24 358.9 mm to (24.8, 153.2)
- moved D1 311.9 mm to (66.7, 113.3), turned to 90 degrees
- moved D2 292.6 mm to (85.7, 113.3), turned to 90 degrees
- moved D3 273.3 mm to (104.8, 113.3), turned to 90 degrees
- moved D4 254.0 mm to (123.8, 113.3), turned to 90 degrees
- moved D5 234.7 mm to (142.9, 113.3), turned to 90 degrees
- moved D6 215.4 mm to (161.9, 113.3), turned to 90 degrees
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Connections:
- net /RF renamed Net-(J3-In)

Commit message: Place all key matrix diodes
Parts:
- D16, D17, D18, D19, D20, D21, D22, D23, D24, D25, D26, D27, D28, D29, D30, D31, D32, D33, D34, D35, D36, D37, D38, D39, D40, D41, D42, D43, D45, D46, D47, D48, D49, D50, D51, D52, D53, D54, D55, D56, D57, D58, D59, D60, D61, D62, D63, D67, D70, D71, D72, D73, D74, D75: moved to B.Cu
- moved D61 335.8 mm to (71.4, 190.0), turned to 90 degrees
- moved D62 329.2 mm to (95.2, 190.0), turned to 90 degrees
- moved D46 328.5 mm to (71.4, 171.0), turned to 90 degrees
- moved D31 311.4 mm to (81.0, 152.0), turned to 90 degrees
- moved D47 309.3 mm to (90.5, 171.0), turned to 90 degrees
- moved D63 306.2 mm to (119.1, 190.0), turned to 90 degrees
- moved D32 292.1 mm to (100.0, 152.0), turned to 90 degrees
- moved D48 290.1 mm to (109.5, 171.0), turned to 90 degrees
- moved D33 272.9 mm to (119.1, 152.0), turned to 90 degrees
- moved D49 271.0 mm to (128.6, 171.0), turned to 90 degrees
- moved D50 269.2 mm to (147.6, 171.0), turned to 90 degrees
- moved D25 257.3 mm to (133.3, 133.0), turned to 90 degrees
- moved D34 253.7 mm to (138.1, 152.0), turned to 90 degrees
- moved D51 250.6 mm to (166.7, 171.0), turned to 90 degrees
- moved D35 234.5 mm to (157.2, 152.0), turned to 90 degrees
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
Commit message: Pick an NTC and calculate R1/R2
Parts:
- moved X1 163.3 mm to (246.3, 85.0)
- moved L1 158.1 mm to (250.0, 89.0), turned to 180 degrees
- moved BT1 79.3 mm to (101.0, 89.0)
- moved U1 29.5 mm to (240.1, 88.5)
- moved J3 27.7 mm to (256.3, 89.0), turned to 180 degrees
Changed lines of the file:
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@@
 	(footprint "Inductor_SMD:L_0805_2012Metric_Pad1.05x1.20mm_HandSolder"
 		(layer "F.Cu")
-		(at 396.95 30.565)
+		(at 250 89 180)
 		(descr "Inductor SMD 0805 (2012 Metric), square (rectangular) end terminal, IPC-7351 nominal with elongated pad for handsoldering. (Body size source: IPC-SM-782 page 80, https://www.pcb-3d.com/wordpress/wp-content/uploads/ipc-sm-782a_amendment_1_and_2.pdf)")
 		(tags "inductor handsolder")
@@
 		(duplicate_pad_numbers_are_jumpers no)
 		(fp_line
-			(start -0.410242 -0.56)
-			(end 0.410242 -0.56)
+			(start -0.410242 0.56)
+			(end 0.410242 0.56)
 			(stroke
 				(width 0.12)
@@
 		)
 		(fp_line
-			(start -0.410242 0.56)
-			(end 0.410242 0.56)
+			(start -0.410242 -0.56)
+			(end 0.410242 -0.56)
 			(stroke
 				(width 0.12)
@@
 		)
 		(pad "1" smd roundrect
-			(at -1.15 0)
+			(at -1.15 0 180)
 			(size 1.05 1.2)
 			(layers "F.Cu" "F.Mask" "F.Paste")
@@
 		)
 		(pad "2" smd roundrect
-			(at 1.15 0)
+			(at 1.15 0 180)
 			(size 1.05 1.2)
 			(layers "F.Cu" "F.Mask" "F.Paste")
@@
 	(footprint "Crystal:Crystal_SMD_2016-4Pin_2.0x1.6mm"
 		(layer "F.Cu")
-		(at 401.43 33.965)
+		(at 246.3 85)
 		(descr "SMD2016/4, Crystal, 2.0x1.6mm package, SMD, http://www.q-crystal.com/upload/5/2015552223166229.pdf")
 		(property "Reference" "X1"
@@
 	(footprint "Connector_Coaxial:SMA_Molex_73251-1153_EdgeMount_Horizontal"
 		(layer "F.Cu")
-		(at 255.5 61.29 -90)
+		(at 256.28 89 180)
 		(descr "Molex SMA RF Connectors, Edge Mount, https://tools.molex.com/pdm_docs/sd/732511150_sd.pdf")
 		(tags "sma edge")
 		(property "Reference" "J3"
-			(at -1.5 7 90)
+			(at -1.5 7 0)
 			(layer "F.SilkS")
 			(effects
@@
 		)
 		(property "Value" "Conn_Coaxial"
-			(at -1.72 -7.11 90)
+			(at -1.72 -7.11 0)
 			(layer "F.Fab")
 			(effects
@@
 		)
 		(property "Datasheet" ""
-			(at 0 0 270)
+			(at 0 0 180)
 			(unlocked yes)
 			(layer "F.Fab")
@@
 		)
 		(property "Description" "coaxial connector (BNC, SMA, SMB, SMC, Cinch/RCA, LEMO, ...)"
-			(at 0 0 270)
+			(at 0 0 180)
 			(unlocked yes)
 			(layer "F.Fab")
@@
 		)
 		(fp_line
-			(start -14.29 6.09)
+			(start 2.71 -6.09)
 			(end 2.71 6.09)
 			(stroke
@@
 		)
 		(fp_line
-			(start -14.29 -6.09)
-			(end -14.29 6.09)
+			(start -14.29 6.09)
+			(end 2.71 6.09)
 			(stroke
 				(width 0.05)
@@
 		)
 		(fp_line
-			(start 2.71 -6.09)
-			(end 2.71 6.09)
+			(start -14.29 -6.09)
+			(end -14.29 6.09)
 			(stroke
 				(width 0.05)
@@
 		)
 		(fp_line
-			(start -14.29 6.09)
+			(start 2.71 -6.09)
 			(end 2.71 6.09)
 			(stroke
@@
 		)
 		(fp_line
-			(start -14.29 -6.09)
-			(end -14.29 6.09)
+			(start 2.71 -6.09)
+			(end -14.29 -6.09)
 			(stroke
 				(width 0.05)
@@
 		)
 		(fp_line
-			(start 2.71 -6.09)
+			(start -14.29 6.09)
 			(end 2.71 6.09)
 			(stroke
@@
 		)
 		(fp_line
-			(start 2.71 -6.09)
-			(end -14.29 -6.09)
+			(start -14.29 -6.09)
+			(end -14.29 6.09)
 			(stroke
 				(width 0.05)
@@
 		)
 		(fp_line
-			(start -5.91 4.76)
+			(start 0.49 3.75)
 			(end 0.49 4.76)
 			(stroke
@@
 		)
 		(fp_line
-			(start -4.76 3.75)
-			(end 0.49 3.75)
+			(start 0.49 -0.38)
+			(end 0.49 0.38)
 			(stroke
 				(width 0.1)
@@
 		)
 		(fp_line
-			(start 0.49 3.75)
-			(end 0.49 4.76)
+			(start 0.49 -4.76)
+			(end 0.49 -3.75)
 			(stroke
 				(width 0.1)
@@
 		)
 		(fp_line
-			(start -13.79 2.65)
-			(end -5.91 2.65)
+			(start 0.49 -4.76)
+			(end -5.91 -4.76)
 			(stroke
 				(width 0.1)
@@
 		)
 		(fp_line
-			(start -4.76 0.38)
-			(end 0.49 0.38)
+			(start -4.76 3.75)
+			(end 0.49 3.75)
 			(stroke
 				(width 0.1)
@@
 		)
 		(fp_line
-			(start -4.76 -0.38)
-			(end 0.49 -0.38)
+			(start -4.76 0.38)
+			(end 0.49 0.38)
 			(stroke
 				(width 0.1)
@@
 		)
 		(fp_line
-			(start 0.49 -0.38)
-			(end 0.49 0.38)
+			(start -4.76 -0.38)
+			(end 0.49 -0.38)
 			(stroke
 				(width 0.1)
@@
 		)
 		(fp_line
-			(start -13.79 -2.65)
-			(end -13.79 2.65)
+			(start -4.76 -3.75)
+			(end 0.49 -3.75)
 			(stroke
 				(width 0.1)
@@
 		)
 		(fp_line
-			(start -13.79 -2.65)
-			(end -5.91 -2.65)
+			(start -4.76 -3.75)
+			(end -4.76 3.75)
 			(stroke
 				(width 0.1)
@@
 		)
 		(fp_line
-			(start -4.76 -3.75)
-			(end -4.76 3.75)
+			(start -5.91 4.76)
+			(end 0.49 4.76)
 			(stroke
 				(width 0.1)
@@
 		)
 		(fp_line
-			(start -4.76 -3.75)
-			(end 0.49 -3.75)
+			(start -5.91 -4.76)
+			(end -5.91 4.76)
 			(stroke
 				(width 0.1)
@@
 		)
 		(fp_line
-			(start -5.91 -4.76)
-			(end -5.91 4.76)
+			(start -13.79 2.65)
+			(end -5.91 2.65)
 			(stroke
 				(width 0.1)
@@
 		)
 		(fp_line
-			(start 0.49 -4.76)
-			(end 0.49 -3.75)
+			(start -13.79 -2.65)
+			(end -5.91 -2.65)
 			(stroke
 				(width 0.1)
@@
 		)
 		(fp_line
-			(start 0.49 -4.76)
-			(end -5.91 -4.76)
+			(start -13.79 -2.65)
+			(end -13.79 2.65)
 			(stroke
 				(width 0.1)
@@
 		)
 		(fp_text user "${REFERENCE}"
-			(at -1.5 7 90)
+			(at -1.5 7 0)
 			(layer "F.Fab")
 			(effects
@@
 		)
 		(pad "1" smd rect
-			(at -1.72 0 270)
+			(at -1.72 0 180)
 			(size 5.08 2.29)
 			(layers "F.Cu" "F.Mask" "F.Paste")
@@
 		)
 		(pad "2" smd rect
-			(at -1.72 -4.38 270)
+			(at -1.72 -4.38 180)
 			(size 5.08 2.42)
 			(layers "F.Cu" "F.Mask" "F.Paste")
@@
 		)
 		(pad "2" smd rect
-			(at -1.72 -4.38 270)
+			(at -1.72 -4.38 180)
 			(size 5.08 2.42)
 			(layers "B.Cu" "B.Mask" "B.Paste")
@@
 		)
 		(pad "2" smd rect
-			(at -1.72 4.38 270)
+			(at -1.72 4.38 180)
 			(size 5.08 2.42)
 			(layers "F.Cu" "F.Mask" "F.Paste")
@@
 		)
 		(pad "2" smd rect
-			(at -1.72 4.38 270)
+			(at -1.72 4.38 180)
 			(size 5.08 2.42)
 			(layers "B.Cu" "B.Mask" "B.Paste")
@@
 		)
 		(pad "2" smd rect
-			(at 1.27 -4.38 270)
+			(at 1.27 -4.38 180)
 			(size 0.95 0.46)
 			(layers "F.Cu")
@@
 		)
 		(pad "2" smd rect
-			(at 1.27 -4.38 270)
+			(at 1.27 -4.38 180)
 			(size 0.95 0.46)
 			(layers "B.Cu")
@@
 		)
 		(pad "2" smd rect
-			(at 1.27 4.38 270)
+			(at 1.27 4.38 180)
 			(size 0.95 0.46)
 			(layers "F.Cu")
@@
 		)
 		(pad "2" smd rect
-			(at 1.27 4.38 270)
+			(at 1.27 4.38 180)
 			(size 0.95 0.46)
 			(layers "B.Cu")
@@
 		)
 		(pad "2" thru_hole circle
-			(at 1.72 -4.38 270)
+			(at 1.72 -4.38 180)
 			(size 0.97 0.97)
 			(drill 0.46)
@@
 		)
 		(pad "2" thru_hole circle
-			(at 1.72 4.38 270)
+			(at 1.72 4.38 180)
 			(size 0.97 0.97)
 			(drill 0.46)
@@
 	(footprint "Package_DFN_QFN:Nordic_AQFN-73-1EP_7x7mm_P0.5mm"
 		(layer "F.Cu")
-		(at 269.2875 83.9675)
+		(at 240.1375 88.5)
 		(descr "http://infocenter.nordicsemi.com/index.jsp?topic=%2Fcom.nordic.infocenter.nrf52%2Fdita%2Fnrf52%2Fchips%2Fnrf52840.html")
 		(tags "AQFN 7mm ")
@@
 	(footprint "Battery:BatteryHolder_Keystone_1042_1x18650"
 		(layer "B.Cu")
-		(at 180.2 85.18 180)
+		(at 100.9675 89 180)
 		(descr "Battery holder, Keystone 1042, battery type 1x18650, http://www.keyelco.com/product.cfm/product_id/918")
 		(tags "horizontal single")

Commit message: idk, moved some bits round?
Parts:
- added TH1: NTC, Resistor_SMD:R_0805_2012Metric_Pad1.20x1.40mm_HandSolder, B.Cu at (153.5, 81.0)
- R12: value R -> 420k
- R13: value R -> 44k
- moved D64 85.3 mm to (240.2, 73.0)
- moved BT1 10.4 mm to (111.4, 89.0)
Changed lines of the file:
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@@
 			)
 		)
-		(property "Value" "R"
+		(property "Value" "44k"
 			(at 0 1.65 0)
 			(layer "F.Fab")
@@
 	(footprint "Diode_SMD:D_SMB_Handsoldering"
 		(layer "F.Cu")
-		(at 317.3 36.5)
+		(at 240.2 73)
 		(descr "Diode SMB (DO-214AA) Handsoldering")
 		(tags "Diode SMB (DO-214AA) Handsoldering")
@@
 			)
 		)
-		(property "Value" "R"
+		(property "Value" "420k"
 			(at 0 1.65 0)
 			(layer "F.Fab")
@@
 		)
 	)
+	(footprint "Resistor_SMD:R_0805_2012Metric_Pad1.20x1.40mm_HandSolder"
+		(layer "B.Cu")
+		(at 153.5 81 -90)
+		(descr "Resistor SMD 0805 (2012 Metric), square (rectangular) end terminal, IPC-7351 nominal with elongated pad for handsoldering. (Body size source: IPC-SM-782 page 72, https://www.pcb-3d.com/wordpress/wp-content/uploads/ipc-sm-782a_amendment_1_and_2.pdf)")
+		(tags "resistor handsolder")
+		(property "Reference" "TH1"
+			(at 0 1.65 90)
+			(layer "B.SilkS")
+			(effects
+				(font
+					(size 1 1)
+					(thickness 0.15)
+				)
+				(justify mirror)
+			)
+		)
+		(property "Value" "NTC"
+			(at 0 -1.65 90)
+			(layer "B.Fab")
+			(effects
+				(font
+					(size 1 1)
+					(thickness 0.15)
+				)
+				(justify mirror)
+			)
+		)
+		(property "Datasheet" ""
+			(at 0 0 90)
+			(layer "B.Fab")
+			(hide yes)
+			(effects
+				(font
+					(size 1.27 1.27)
+				)
+				(justify mirror)
+			)
+		)
+		(property "Description" "Temperature dependent resistor, negative temperature coefficient"
+			(at 0 0 90)
+			(layer "B.Fab")
+			(hide yes)
+			(effects
+				(font
+					(size 1.27 1.27)
+				)
+				(justify mirror)
+			)
+		)
+		(property "KiLib_Generator" "SMD_2terminal_chip_molded"
+			(at 0 0 90)
+			(layer "B.SilkS")
+			(hide yes)
+			(effects
+				(font
+					(size 1 1)
+					(thickness 0.15)
+				)
+				(justify mirror)
+			)
+		)
+		(property ki_fp_filters "R_* RV_*")
+		(sheetname "/power/")
+		(sheetfile "usb.kicad_sch")
+		(units
+			(unit
+				(name "A")
+				(pins "1" "2")
+			)
+		)
+		(attr smd)
+		(duplicate_pad_numbers_are_jumpers no)
+		(fp_line
+			(start -0.227064 0.735)
+			(end 0.227064 0.735)
+			(stroke
+				(width 0.12)
+				(type solid)
+			)
+			(layer "B.SilkS")
+		)
+		(fp_line
+			(start -0.227064 -0.735)
+			(end 0.227064 -0.735)
+			(stroke
+				(width 0.12)
+				(type solid)
+			)
+			(layer "B.SilkS")
+		)
+		(fp_rect
+			(start -1.85 0.95)
+			(end 1.85 -0.95)
+			(stroke
+				(width 0.05)
+				(type solid)
+			)
+			(fill no)
+			(layer "B.CrtYd")
+		)
+		(fp_rect
+			(start -1 0.625)
+			(end 1 -0.625)
+			(stroke
+				(width 0.1)
+				(type solid)
+			)
+			(fill no)
+			(layer "B.Fab")
+		)
+		(fp_text user "${REFERENCE}"
+			(at 0 0 90)
+			(layer "B.Fab")
+			(effects
+				(font
+					(size 0.5 0.5)
+					(thickness 0.08)
+				)
+				(justify mirror)
+			)
+		)
+		(pad "1" smd roundrect
+			(at -1 0 270)
+			(size 1.2 1.4)
+			(layers "B.Cu" "B.Mask" "B.Paste")
+			(roundrect_rratio 0.208333)
+			(net "Net-(U2-TEMP)")
+			(pintype "passive")
+		)
+		(pad "2" smd roundrect
+			(at 1 0 270)
+			(size 1.2 1.4)
+			(layers "B.Cu" "B.Mask" "B.Paste")
+			(roundrect_rratio 0.208333)
+			(net "GND")
+			(pintype "passive")
+		)
+		(embedded_fonts no)
+		(model "${KICAD10_3DMODEL_DIR}/Resistor_SMD.3dshapes/R_0805_2012Metric.step"
+			(offset
+				(xyz 0 0 0)
+			)
+			(scale
+				(xyz 1 1 1)
+			)
+			(rotate
+				(xyz 0 0 0)
+			)
+		)
+	)
 	(footprint "Diode_SMD:D_0805_2012Metric_Pad1.15x1.40mm_HandSolder"
 		(layer "B.Cu")
@@
 	(footprint "Battery:BatteryHolder_Keystone_1042_1x18650"
 		(layer "B.Cu")
-		(at 100.9675 89 180)
+		(at 111.38 89 180)
 		(descr "Battery holder, Keystone 1042, battery type 1x18650, http://www.keyelco.com/product.cfm/product_id/918")
 		(tags "horizontal single")

Commit message: Did a bunch of stuff lol
Parts:
- added J1: Conn_ARM_JTAG_SWD_10, Connector_IDC:IDC-Header_2x05_P2.54mm_Vertical, F.Cu at (205.9, 93.2)
- added J2: USB_C_Receptacle_USB2.0_16P, My_Footprints:USB_C_Receptacle_G-Switch_GT-USB-7010ASV_handsolder_lmao.csv, F.Cu at (66.8, 80.4)
- added SW1: SW_SPST, My_Footprints:Legion SS11, F.Cu at (175.2, 88.1)
- added SW2: SW_SPST, My_Footprints:Legion SS11, F.Cu at (190.9, 88.1)
- BT1, TH1: moved to F.Cu
- C1, C10, C12, C13, C14, C15, C16, C17, C18, C19, C2, C20, C21, C22, C3, C4, C5, C6, C7, C8, C9: footprint Capacitor_SMD:C_0805_2012Metric_Pad1.18x1.45mm_HandSolder -> Capacitor_SMD:C_0603_1608Metric_Pad1.08x0.95mm_HandSolder
- L1, L2, L3: footprint Inductor_SMD:L_0805_2012Metric_Pad1.05x1.20mm_HandSolder -> Inductor_SMD:L_0603_1608Metric_Pad1.05x0.95mm_HandSolder
- moved D44 288.2 mm to (67.0, 90.2), turned to 180 degrees
- moved R2 232.5 mm to (63.2, 90.1), turned to -90 degrees
- moved R1 225.9 mm to (70.5, 90.0), turned to -90 degrees
- moved C20 175.6 mm to (231.4, 97.4), turned to -90 degrees
- moved L2 174.8 mm to (229.5, 83.6), turned to -90 degrees
- moved L3 173.1 mm to (229.5, 79.8), turned to -90 degrees
- moved C16 170.9 mm to (232.5, 81.9)
- moved C5 165.6 mm to (226.3, 87.9), turned to 180 degrees
- moved C15 161.2 mm to (232.5, 83.7)
- moved C13 160.1 mm to (235.5, 83.5), turned to 90 degrees
- moved C9 159.9 mm to (240.3, 86.6)
- moved C1 157.8 mm to (237.7, 83.5), turned to -90 degrees
- moved C3 153.5 mm to (243.5, 91.9), turned to -90 degrees
- moved C22 152.0 mm to (252.1, 91.9), turned to -90 degrees
- moved C10 152.0 mm to (247.1, 85.4)
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Other:
- board outline added: 304.8 x 119.1 mm
