File: pcb/keyboard.kicad_pcb (KiCad board)
At the start: 4 copper layers, 304.8 x 119.1 mm, 208 parts, among them J1 Conn_ARM_JTAG_SWD_10, J2 USB_C_Receptacle_USB2.0_16P, J3 Conn_Coaxial, K1 KEYSW, K10 KEYSW, K11 KEYSW, K12 KEYSW, K13 KEYSW, K14 KEYSW, K15 KEYSW, K16 KEYSW, K17 KEYSW, K18 KEYSW, K19 KEYSW, K2 KEYSW, K20 KEYSW, K21 KEYSW, K22 KEYSW, K23 KEYSW, K24 KEYSW, K25 KEYSW, K26 KEYSW, K27 KEYSW, K28 KEYSW, K29 KEYSW, K3 KEYSW, K30 KEYSW, K31 KEYSW, K32 KEYSW, K33 KEYSW, K34 KEYSW, K35 KEYSW, K36 KEYSW, K37 KEYSW, K38 KEYSW, K39 KEYSW, K4 KEYSW, K40 KEYSW, K41 KEYSW, K42 KEYSW, K43 KEYSW, K45 KEYSW, K46 KEYSW, K47 KEYSW, K48 KEYSW, K49 KEYSW, K5 KEYSW, K50 KEYSW, K51 KEYSW, K52 KEYSW, K53 KEYSW, K54 KEYSW, K55 KEYSW, K56 KEYSW, K57 KEYSW, K58 KEYSW, K59 KEYSW, K6 KEYSW, K60 KEYSW, K61 KEYSW, K62 KEYSW, K63 KEYSW, K67 KEYSW, K7 KEYSW, K70 KEYSW, K71 KEYSW, K72 KEYSW, K73 KEYSW, K74 KEYSW, K75 KEYSW, K8 KEYSW, K9 KEYSW, Q1 FDN340P, Q2 FS8025A, Q3 FDN340P, SW1 SW_SPST, SW2 SW_SPST, U1 nRF52840, U2 TP4056-42-ESOP8, U3 DW01A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

Commit message: Address initial comments
Parts:
- moved C1 1.52 mm to (238.5, 79.8), turned to -135 degrees
- moved C15 1.00 mm to (230.0, 82.0)
- moved C16 1.00 mm to (230.0, 80.0)
- moved L2 0.50 mm to (226.5, 82.0)
- moved L3 0.50 mm to (226.5, 80.0)
Routing:
- net GND: track 70.6 -> 78.4 mm
- net col0: track 273.5 -> 272.4 mm
- net VBUS: track 15.3 -> 15.8 mm
Other:
- board text removed: "TODO: Move vias from overlapping with silkscreen"

Commit message: Address DRC violations
Routing:
- net /DEC4_6: track 19.1 -> 40.3 mm
- net GND: track 78.4 -> 82.3 mm, vias 43 -> 40
- net row1: track 366.1 -> 366.0 mm, vias 18 -> 17
- net row0: vias 18 -> 19

Commit message: Fuck around with silkscreen stuff
Parts:
- added G***: LOGO, My_Footprints:pfp, F.Cu at (54.5, 93.5)
- K1, K10, K11, K12, K13, K15, K17, K18, K19, K2, K20, K21, K22, K23, K24, K25, K26, K27, K28, K3, K30, K32, K33, K34, K35, K36, K37, K38, K39, K4, K40, K41, K42, K43, K45, K47, K48, K49, K5, K50, K51, K52, K53, K54, K55, K56, K57, K59, K6, K60, K7, K70, K71, K72, K73, K74, K75, K8, K9: footprint Switch_Keyboard_Hotswap_Kailh:SW_Hotswap_Kailh_MX_1.00u -> My_Footprints:SW_Hotswap_Kailh_MX_1.00u
- K16: footprint Switch_Keyboard_Hotswap_Kailh:SW_Hotswap_Kailh_MX_1.50u -> My_Footprints:SW_Hotswap_Kailh_MX_1.25u
- K31, K58: footprint Switch_Keyboard_Hotswap_Kailh:SW_Hotswap_Kailh_MX_1.75u -> My_Footprints:SW_Hotswap_Kailh_MX_1.75u
- K46, K61, K62, K63: footprint Switch_Keyboard_Hotswap_Kailh:SW_Hotswap_Kailh_MX_1.25u -> My_Footprints:SW_Hotswap_Kailh_MX_1.25u
